Commit message: new

File: rotors_gazebo/models/rotors_description/urdf/multirotor_base.xacro (robot description, xacro)
@@ -56,5 +56,5 @@
     </gazebo>
     <gazebo reference="base_link">
-      <material>Gazebo/${color}</material>
+      <material>Gazebo/DarkGray</material>
       <collision name='base_link_inertia_collision'>
         <surface>
